File: catt_rs485.kicad_sch (KiCad schematic)
At the start: 22 parts, among them J1 CATT, J2 Output, U3 24C02BN, U4 SN65HVD75DR, U5 SN65HVD75DR

Commit message: Renumber components
Parts:
- renumbered C2 to C1, C4 to C2, C5 to C3, C3 to C4, D6 to D1, D7 to D2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

Commit message: Add missing LCSC number of output connector
Parts:
- J2: LCSC (none) -> C7246
Changed lines of the file:
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@@
+			)
+		)
+		(property "LCSC" "C7246"
+			(at 254 138.43 0)
+			(effects
+				(font
+					(size 1.27 1.27)
+				)
+				(hide yes)
 			)
 		)
